File: electronics/controllino-can.kicad_pcb (KiCad board)
At the start: 2 copper layers, 19.2 x 34 mm, 12 parts, among them J2 Conn_02x13_Odd_Even, J5 TBL002A-350-04GR-2OR, U1 MCP2515-xST, U2 MCP2562-E-SN, Y2 8 MHz

Commit message: updated pcb silkscreen and added pcb render. Also added BOM for digikey
Parts:
- added kibuzzard-653F042B: G***, kibuzzard-653F042B, B.Cu at (79.0, 47.5)
- added kibuzzard-653F0443: G***, kibuzzard-653F0443, B.Cu at (75.9, 43.9)
- added kibuzzard-653F047F: G***, kibuzzard-653F047F, B.Cu at (79.2, 54.4)
- added kibuzzard-653F0498: G***, kibuzzard-653F0498, B.Cu at (75.4, 50.8)
Other:
- board text added: "5V+"
- board text added: "CANH"
- board text added: "CANL"
- board text added: "GND"
- board text added: "TERMINATING RESISTOR"
- board text removed: "G"
- board text removed: "H"
- board text removed: "L"
